File: schematic/schematic/schematic.sch (KiCad schematic (older format))
At the start: 105 parts, among them J1 USB_A, J10 Conn_Tale, J2 USB_B_Micro, J3 Conn_PWM0, J4 Conn_PWM1, J5 Conn_SPI, J6 Conn_I2C, J7 Conn_GPIO, J8 Conn_Tale, J9 Conn_M5StickV, M1 Motor_DC, Q1 SS8050, Q2 SS8050, Q3 IRLML6402, Q4 PJE260N02, Q5 IRLML6402, Q6 PJE260N02, Q7 PJE260N02, SW1 SW_EN, SW2 SW_IO0, SW3 PS-85N, U1 TPS63002, U2 TPS63001, U3 MCP73831-5-OT, U4 FT231XS, U5 DW01-P, U6 BR8205, U7 TB6612FNG, U8 ESP32-WROOM-32D

Commit message: assign footprint
Parts:
- D1, D4: footprint (none) -> Diode_SMD:D_SOD-123F
- D10, D2, D5, D6, D8, D9: footprint (none) -> LED_SMD:LED_0603_1608Metric_Pad1.05x0.95mm_HandSolder
- D7: footprint (none) -> micelib:LTSN-B32JEGBB6
- F1: footprint (none) -> Resistor_SMD:R_1812_4532Metric_Pad1.30x3.40mm_HandSolder
- J10, J5, J8: footprint (none) -> Connector_PinHeader_2.54mm:PinHeader_1x05_P2.54mm_Vertical
- J3, J4: footprint (none) -> Connector_PinHeader_2.54mm:PinHeader_1x03_P2.54mm_Vertical
- J6: footprint (none) -> Connector_PinHeader_2.54mm:PinHeader_1x04_P2.54mm_Vertical
- J7: footprint (none) -> Connector_PinHeader_2.54mm:PinHeader_1x02_P2.54mm_Vertical
- J9: footprint (none) -> Connector_PinSocket_2.54mm:PinSocket_1x04_P2.54mm_Vertical
- JP1, JP2: footprint (none) -> Jumper:SolderJumper-2_P1.3mm_Bridged2Bar_Pad1.0x1.5mm
- Q1, Q2, Q3, Q5: footprint (none) -> Package_TO_SOT_SMD:SOT-23
- Q4, Q6, Q7: footprint (none) -> Package_TO_SOT_SMD:SOT-416
- SW1, SW2: footprint (none) -> micelib:SW_SPST_PTS810_HandSoldering
- SW3: footprint (none) -> micelib:PS-85
- U1: footprint micelib:WSON-10-1EP_2x3mm_P0.5mm_EP0.84x2.4mm_TPS6300x -> Connector_PinHeader_2.54mm:PinHeader_1x05_P2.54mm_Vertical
- U5, U6: footprint (none) -> Package_TO_SOT_SMD:SOT-23-6_Handsoldering
Changed lines of the file:
@@
 F 0 "J9" H 9800 5850 50  0000 L CNN
 F 1 "Conn_M5StickV" H 9200 5600 50  0000 L CNN
-F 2 "" H 9700 5900 50  0001 C CNN
+F 2 "Connector_PinSocket_2.54mm:PinSocket_1x04_P2.54mm_Vertical" H 9700 5900 50  0001 C CNN
 F 3 "~" H 9700 5900 50  0001 C CNN
 	1    9700 5900
@@
 F 0 "Q5" V 6543 7300 50  0000 C CNN
 F 1 "IRLML6402" V 6452 7300 50  0000 C CNN
-F 2 "" H 6400 7400 50  0001 C CNN
+F 2 "Package_TO_SOT_SMD:SOT-23" H 6400 7400 50  0001 C CNN
 F 3 "~" H 6200 7300 50  0001 C CNN
 	1    6200 7300
@@
 F 0 "U1" H 1600 3865 50  0000 C CNN
 F 1 "TPS63002" H 1600 3774 50  0000 C CNN
-F 2 "micelib:WSON-10-1EP_2x3mm_P0.5mm_EP0.84x2.4mm_TPS6300x" H 1600 3400 50  0001 C CNN
+F 2 "Connector_PinHeader_2.54mm:PinHeader_1x05_P2.54mm_Vertical" H 1600 3400 50  0001 C CNN
 F 3 "" H 1600 3400 50  0001 C CNN
 	1    1600 3400
@@
 F 0 "U5" H 4450 6215 50  0000 C CNN
 F 1 "DW01-P" H 4450 6124 50  0000 C CNN
-F 2 "" H 4450 5850 50  0001 C CNN
+F 2 "Package_TO_SOT_SMD:SOT-23-6_Handsoldering" H 4450 5850 50  0001 C CNN
 F 3 "" H 4450 5850 50  0001 C CNN
 	1    4450 5850
@@
 F 0 "U6" H 4450 7315 50  0000 C CNN
 F 1 "BR8205" H 4450 7224 50  0000 C CNN
-F 2 "" H 4450 6950 50  0001 C CNN
+F 2 "Package_TO_SOT_SMD:SOT-23-6_Handsoldering" H 4450 6950 50  0001 C CNN
 F 3 "" H 4450 6950 50  0001 C CNN
 	1    4450 6950
@@
 F 0 "D9" V 8000 1100 50  0000 R CNN
 F 1 "LED_Charge" V 7900 1400 50  0000 R CNN
-F 2 "" V 7950 900 50  0001 C CNN
+F 2 "LED_SMD:LED_0603_1608Metric_Pad1.05x0.95mm_HandSolder" V 7950 900 50  0001 C CNN
 F 3 "~" V 7950 900 50  0001 C CNN
 	1    7950 900
@@
 F 0 "Q3" V 5700 5800 50  0000 C CNN
 F 1 "IRLML6402" V 5650 5500 50  0000 C CNN
-F 2 "" H 5650 5900 50  0001 C CNN
+F 2 "Package_TO_SOT_SMD:SOT-23" H 5650 5900 50  0001 C CNN
 F 3 "~" H 5450 5800 50  0001 C CNN
 	1    5450 5800
@@
 F 0 "D4" H 6300 5550 50  0000 R CNN
 F 1 "SS2040FL" H 6250 5700 50  0000 R CNN
-F 2 "" V 6150 5600 50  0001 C CNN
+F 2 "Diode_SMD:D_SOD-123F" V 6150 5600 50  0001 C CNN
 F 3 "~" V 6150 5600 50  0001 C CNN
 	1    6150 5600
@@
 F 0 "SW3" H 5450 6950 60  0000 C CNN
 F 1 "PS-85N" H 5400 7300 60  0000 C CNN
-F 2 "" H 5450 6950 60  0001 C CNN
+F 2 "micelib:PS-85" H 5450 6950 60  0001 C CNN
 F 3 "" H 5450 6950 60  0001 C CNN
 	1    5450 6950
@@
 F 0 "SW1" V 3054 1298 50  0000 L CNN
 F 1 "SW_EN" V 3145 1298 50  0000 L CNN
-F 2 "" H 3100 1350 50  0001 C CNN
+F 2 "micelib:SW_SPST_PTS810_HandSoldering" H 3100 1350 50  0001 C CNN
 F 3 "" H 3100 1350 50  0001 C CNN
 	1    3100 1150
@@
 F 0 "SW2" V 3604 1298 50  0000 L CNN
 F 1 "SW_IO0" V 3695 1298 50  0000 L CNN
-F 2 "" H 3650 1350 50  0001 C CNN
+F 2 "micelib:SW_SPST_PTS810_HandSoldering" H 3650 1350 50  0001 C CNN
 F 3 "" H 3650 1350 50  0001 C CNN
 	1    3650 1150
@@
 F 0 "Q1" H 5141 1046 50  0000 L CNN
 F 1 "SS8050" H 5141 955 50  0000 L CNN
-F 2 "" H 5150 1100 50  0001 C CNN
+F 2 "Package_TO_SOT_SMD:SOT-23" H 5150 1100 50  0001 C CNN
 F 3 "~" H 4950 1000 50  0001 C CNN
 	1    4950 1000
@@
 F 0 "Q2" H 5141 1604 50  0000 L CNN
 F 1 "SS8050" H 5141 1695 50  0000 L CNN
-F 2 "" H 5150 1750 50  0001 C CNN
+F 2 "Package_TO_SOT_SMD:SOT-23" H 5150 1750 50  0001 C CNN
 F 3 "~" H 4950 1650 50  0001 C CNN
 	1    4950 1650
@@
 F 0 "JP1" H 2000 3950 50  0000 C CNN
 F 1 "Jumper" H 2000 3800 50  0000 C CNN
-F 2 "" H 2000 3850 50  0001 C CNN
+F 2 "Jumper:SolderJumper-2_P1.3mm_Bridged2Bar_Pad1.0x1.5mm" H 2000 3850 50  0001 C CNN
 F 3 "~" H 2000 3850 50  0001 C CNN
 	1    2000 3850
@@
 F 0 "JP2" H 2050 2250 50  0000 C CNN
 F 1 "Jumper" H 2050 2100 50  0000 C CNN
-F 2 "" H 2050 2150 50  0001 C CNN
+F 2 "Jumper:SolderJumper-2_P1.3mm_Bridged2Bar_Pad1.0x1.5mm" H 2050 2150 50  0001 C CNN
 F 3 "~" H 2050 2150 50  0001 C CNN
 	1    2050 2150
@@
 F 0 "D6" V 6446 1832 50  0000 R CNN
 F 1 "LED_5V" V 6355 1832 50  0000 R CNN
-F 2 "" V 6400 1900 50  0001 C CNN
+F 2 "LED_SMD:LED_0603_1608Metric_Pad1.05x0.95mm_HandSolder" V 6400 1900 50  0001 C CNN
 F 3 "~" V 6400 1900 50  0001 C CNN
 	1    6400 1900
@@
 F 0 "D7" H 6600 1000 50  0000 L CNN
 F 1 "LTSN-B32JEGBB6" H 6300 1400 50  0000 L CNN
-F 2 "" H 6650 1200 50  0001 C CNN
+F 2 "micelib:LTSN-B32JEGBB6" H 6650 1200 50  0001 C CNN
 F 3 "" H 6650 1200 50  0001 C CNN
 	1    6650 1200
@@
 F 0 "J6" H 5230 4492 50  0000 L CNN
 F 1 "Conn_I2C" H 4950 4200 50  0000 L CNN
-F 2 "" H 5150 4500 50  0001 C CNN
+F 2 "Connector_PinHeader_2.54mm:PinHeader_1x04_P2.54mm_Vertical" H 5150 4500 50  0001 C CNN
 F 3 "~" H 5150 4500 50  0001 C CNN
 	1    5150 4500
@@
 F 0 "J3" H 2029 4642 50  0000 L CNN
 F 1 "Conn_PWM0" H 1750 4400 50  0000 L CNN
-F 2 "" H 1950 4600 50  0001 C CNN
+F 2 "Connector_PinHeader_2.54mm:PinHeader_1x03_P2.54mm_Vertical" H 1950 4600 50  0001 C CNN
 F 3 "~" H 1950 4600 50  0001 C CNN
 	1    1950 4600
@@
 F 0 "J4" H 2929 4642 50  0000 L CNN
 F 1 "Conn_PWM1" H 2650 4400 50  0000 L CNN
-F 2 "" H 2850 4600 50  0001 C CNN
+F 2 "Connector_PinHeader_2.54mm:PinHeader_1x03_P2.54mm_Vertical" H 2850 4600 50  0001 C CNN
 F 3 "~" H 2850 4600 50  0001 C CNN
 	1    2850 4600
@@
 F 0 "D2" V 5846 2882 50  0000 R CNN
 F 1 "LED_Brake" V 5755 2882 50  0000 R CNN
-F 2 "" V 5800 2950 50  0001 C CNN
+F 2 "LED_SMD:LED_0603_1608Metric_Pad1.05x0.95mm_HandSolder" V 5800 2950 50  0001 C CNN
 F 3 "~" V 5800 2950 50  0001 C CNN
 	1    5800 2950
@@
 F 0 "D5" V 6396 2882 50  0000 R CNN
 F 1 "LED_Brake" V 6305 2882 50  0000 R CNN
-F 2 "" V 6350 2950 50  0001 C CNN
+F 2 "LED_SMD:LED_0603_1608Metric_Pad1.05x0.95mm_HandSolder" V 6350 2950 50  0001 C CNN
 F 3 "~" V 6350 2950 50  0001 C CNN
 	1    6350 2950
@@
 F 0 "Q4" H 5750 3700 50  0000 L CNN
 F 1 "PJE260N02" H 5500 3800 50  0000 L CNN
-F 2 "" H 6100 3700 50  0001 C CNN
+F 2 "Package_TO_SOT_SMD:SOT-416" H 6100 3700 50  0001 C CNN
 F 3 "~" H 5900 3600 50  0001 C CNN
 	1    5900 3600
@@
 F 0 "D8" V 6946 2782 50  0000 R CNN
 F 1 "LED_Right" V 6855 2782 50  0000 R CNN
-F 2 "" V 6900 2850 50  0001 C CNN
+F 2 "LED_SMD:LED_0603_1608Metric_Pad1.05x0.95mm_HandSolder" V 6900 2850 50  0001 C CNN
 F 3 "~" V 6900 2850 50  0001 C CNN
 	1    6900 2850
@@
 F 0 "Q6" H 6850 3600 50  0000 L CNN
 F 1 "PJE260N02" H 6600 3700 50  0000 L CNN
-F 2 "" H 7200 3600 50  0001 C CNN
+F 2 "Package_TO_SOT_SMD:SOT-416" H 7200 3600 50  0001 C CNN
 F 3 "~" H 7000 3500 50  0001 C CNN
 	1    7000 3500
@@
 F 0 "D10" V 8046 1732 50  0000 R CNN
 F 1 "LED_Left" V 7955 1732 50  0000 R CNN
-F 2 "" V 8000 1800 50  0001 C CNN
+F 2 "LED_SMD:LED_0603_1608Metric_Pad1.05x0.95mm_HandSolder" V 8000 1800 50  0001 C CNN
 F 3 "~" V 8000 1800 50  0001 C CNN
 	1    8000 1800
@@
 F 0 "Q7" H 7750 2550 50  0000 L CNN
 F 1 "PJE260N02" H 7500 2650 50  0000 L CNN
-F 2 "" H 8100 2550 50  0001 C CNN
+F 2 "Package_TO_SOT_SMD:SOT-416" H 8100 2550 50  0001 C CNN
 F 3 "~" H 7900 2450 50  0001 C CNN
 	1    7900 2450
@@
 F 0 "J10" H 9500 5050 50  0000 L CNN
 F 1 "Conn_Tale" H 9400 5150 50  0000 L CNN
-F 2 "" H 9750 4800 50  0001 C CNN
+F 2 "Connector_PinHeader_2.54mm:PinHeader_1x05_P2.54mm_Vertical" H 9750 4800 50  0001 C CNN
 F 3 "~" H 9750 4800 50  0001 C CNN
 	1    9750 4800
@@
 F 0 "F1" H 5968 6596 50  0000 L CNN
 F 1 "SMD1812P125TS" H 5968 6505 50  0000 L CNN
-F 2 "" H 5950 6350 50  0001 L CNN
+F 2 "Resistor_SMD:R_1812_4532Metric_Pad1.30x3.40mm_HandSolder" H 5950 6350 50  0001 L CNN
 F 3 "~" H 5900 6550 50  0001 C CNN
 	1    5900 6550
@@
 F 0 "D1" H 1300 4855 50  0000 C CNN
 F 1 "SS2040FL" H 1300 4764 50  0000 C CNN
-F 2 "" V 1300 4650 50  0001 C CNN
+F 2 "Diode_SMD:D_SOD-123F" V 1300 4650 50  0001 C CNN
 F 3 "~" V 1300 4650 50  0001 C CNN
 	1    1300 4650
@@
 F 0 "J5" V 4366 4212 50  0000 R CNN
 F 1 "Conn_SPI" V 4500 4750 50  0000 R CNN
-F 2 "" H 4400 4500 50  0001 C CNN
+F 2 "Connector_PinHeader_2.54mm:PinHeader_1x05_P2.54mm_Vertical" H 4400 4500 50  0001 C CNN
 F 3 "~" H 4400 4500 50  0001 C CNN
 	1    4400 4500
@@
 F 0 "J7" H 8370 3175 50  0000 C CNN
 F 1 "Conn_GPIO" H 8350 3250 50  0000 C CNN
-F 2 "" H 8450 3500 50  0001 C CNN
+F 2 "Connector_PinHeader_2.54mm:PinHeader_1x02_P2.54mm_Vertical" H 8450 3500 50  0001 C CNN
 F 3 "~" H 8450 3500 50  0001 C CNN
 	1    8450 3500
@@
 F 0 "J8" H 10100 5050 50  0000 L CNN
 F 1 "Conn_Tale" H 10000 5150 50  0000 L CNN
-F 2 "" H 10350 4800 50  0001 C CNN
+F 2 "Connector_PinHeader_2.54mm:PinHeader_1x05_P2.54mm_Vertical" H 10350 4800 50  0001 C CNN
 F 3 "~" H 10350 4800 50  0001 C CNN
 	1    10350 4800
