File: schematic/schematic/schematic.sch (KiCad schematic (older format))
At the start: 95 parts, among them IC1 DRV8830, J1 USB_B_Micro, J2 Conn_PWM, J3 Conn_GPIO, J4 Conn_M5StickV, J5 Conn_Tale, J6 Conn_Tale, M1 M_Small, Q1 SS8050, Q2 SS8050, Q3 IRLML6402, Q4 PJE260N02, Q5 IRLML6402, Q6 PJE260N02, Q7 BSS138, Q8 BSS138, Q9 PJE260N02, SW1 SW_EN, SW2 SW_IO0, SW3 SW_SPDT, U1 TPS63002, U2 TPS63001, U3 MCP73831-5-OT, U4 FT231XS, U5 DW01-P, U6 BR8205, U7 ESP32-WROOM-32D

Commit message: やっぱり機能を絞るに限る
Parts:
- removed JP1: Jumper, Jumper:SolderJumper-2_P1.3mm_Bridged2Bar_Pad1.0x1.5mm, symbol Device:Jumper_NC_Small
- removed U7: ESP32-WROOM-32D, micelib:ESP32-WROOM-32_Hand, symbol RF_Module:ESP32-WROOM-32D
- added JP1: Jumper_NO_Small, Jumper:SolderJumper-2_P1.3mm_Open_TrianglePad1.0x1.5mm, symbol Device:Jumper_NO_Small
- added U7: ESP32-WROOM-32D_GND_39, micelib:ESP32-WROOM-32_Hand, symbol micelib:ESP32-WROOM-32D_GND_39
- J5: footprint Connector_PinHeader_2.54mm:PinHeader_1x05_P2.54mm_Vertical -> Connector_PinHeader_1.27mm:PinHeader_1x05_P1.27mm_Vertical
Connections:
- net +3V3: now also U7.2 (VDD)
- net +5V: now also R20.1; no longer D7.2 (A)
- net ADC1_Batt: now also U7.7 (IO35)
- net EN: now also U7.3 (EN)
- net ESP32_RX: now also J4.4 (Pin_4), U7.27 (IO16); no longer J4.3 (Pin_3)
- net ESP32_TX: now also J4.3 (Pin_3), U7.28 (IO17); no longer J4.4 (Pin_4)
- net FAULTn: now also D7.1 (K); no longer R20.2
- net GND: now also JP1.1; no longer C1.2, C16.1, C17.2, C2.2, C3.2, C6.2, IC1.7 (A0), IC1.8 (A1), J1.5 (GND), J1.6 (Shield), R1.2, R10.2, R7.1, R9.2, SW3.1 (A), U1.11 (GND), U1.3 (PGND), U2.11 (GND), U2.3 (PGND), U3.2 (VSS)
- net GNDD: now also C1.2, C16.1, C17.2, C2.2, C3.2, C6.2, IC1.7 (A0), IC1.8 (A1), J1.5 (GND), J1.6 (Shield), R1.2, R10.2, R7.1, R9.2, SW3.1 (A), U1.11 (GND), U1.3 (PGND), U2.11 (GND), U2.3 (PGND), U3.2 (VSS), JP1.2, U7.1 (GND), U7.15 (GND), U7.38 (GND), U7.39 (GND_PAD)
- net GPIO_18: now also U7.30 (IO18)
- net GPIO_19: now also U7.31 (IO19)
- net GPIO_5: now also U7.29 (IO5)
- net I2C_SCL: now also U7.36 (IO22)
- net I2C_SDA: now also U7.33 (IO21)
- net IO0: now also U7.25 (IO0)
- net LED_BRAKE: now also U7.11 (IO26)
- net LED_LEFT: now also J5.3 (Pin_3), J6.3 (Pin_3), U7.10 (IO25); no longer J5.1 (Pin_1), J6.1 (Pin_1)
- net LED_RIGHT: now also J5.1 (Pin_1), J6.1 (Pin_1), U7.12 (IO27); no longer J5.3 (Pin_3), J6.3 (Pin_3)
- net PWM0: now also J2.2 (Pin_2), U7.8 (IO32); no longer J2.1 (Pin_1)
- net PWM1: now also J2.1 (Pin_1), U7.9 (IO33); no longer J2.2 (Pin_2)
- net SPI_CLK: now also U7.13 (IO14)
- net SPI_MISO: now also U7.14 (IO12)
- net SPI_MOSI: now also U7.16 (IO13)
- net STAT: now also D8.1 (K); no longer R24.2
- net UART_RX: now also U7.34 (RXD0/IO3)
- net UART_TX: now also U7.35 (TXD0/IO1)
- net VBUS: now also R24.1; no longer D8.2 (A)
- net at R37.2: now also U7.23 (IO15)
- net at R32.2: now also U7.24 (IO2)
- new net: D8.2 (A), R24.2
- new net: D7.2 (A), R20.2
Other:
- moved on the sheet: D7, D8, J3, R20, R24
