File: schematic/schematic/schematic.sch (KiCad schematic (older format))
At the start: 95 parts, among them IC1 DRV8830, J1 USB_B_Micro, J2 Conn_PWM, J3 Conn_GPIO, J4 Conn_M5StickV, J5 Conn_Tale, J6 Conn_Tale, M1 M_Small, Q1 SS8050, Q2 SS8050, Q3 IRLML6402, Q4 PJE260N02, Q5 IRLML6402, Q6 PJE260N02, Q7 BSS138, Q8 BSS138, Q9 PJE260N02, SW1 SW_EN, SW2 SW_IO0, SW3 SW_SPDT, U1 TPS63002, U2 TPS63001, U3 MCP73831-5-OT, U4 FT231XS, U5 DW01-P, U6 BR8205, U7 ESP32-WROOM-32D_GND_39

Commit message: Update Board
Parts:
- removed C11: 0.1u, micelib:C_0402_1005Metric_HandSoldering, symbol Device:C_Small
- removed C2, C5: 10u, Capacitor_SMD:C_0603_1608Metric_Pad1.05x0.95mm_HandSolder, symbol Device:C_Small
- removed D8: LED_Charge, LED_SMD:LED_0603_1608Metric_Pad1.05x0.95mm_HandSolder, symbol Device:LED_Small
- removed J2: Conn_PWM, Connector_PinSocket_2.54mm:PinSocket_2x03_P2.54mm_Vertical, symbol Connector_Generic:Conn_02x03_Odd_Even
- removed L2: 2.2u, micelib:SPM3015-xRxM-LR, symbol Device:L_Small
- removed R24, R9: 1k, micelib:C_0402_1005Metric_HandSoldering, symbol Device:R_Small
- removed R4: 100, micelib:C_0402_1005Metric_HandSoldering, symbol Device:R_Small
- removed R7: 0.1, Resistor_SMD:R_1206_3216Metric_Pad1.42x1.75mm_HandSolder, symbol Device:R_Small
- removed TP1: VBAT, Connector_PinHeader_1.27mm:PinHeader_1x01_P1.27mm_Vertical, symbol Connector:TestPoint
- removed TP2: -VBAT, Connector_PinHeader_1.27mm:PinHeader_1x01_P1.27mm_Vertical, symbol Connector:TestPoint
- removed TP3: +BATT, Connector_PinHeader_1.27mm:PinHeader_1x01_P1.27mm_Vertical, symbol Connector:TestPoint
- removed U2: TPS63001, micelib:WSON-10-1EP_2x3mm_P0.5mm_EP0.84x2.4mm_TPS6300x, symbol micelib:TPS6300x
- removed U5: DW01-P, Package_TO_SOT_SMD:SOT-23-6_Handsoldering, symbol micelib:DW01-P
- removed U6: BR8205, Package_TO_SOT_SMD:SOT-23-6_Handsoldering, symbol micelib:BR8205
- added C? (x3): 0.1u, micelib:C_0402_1005Metric_HandSoldering, symbol Device:C_Small
- added C? (x2): 0.1u, symbol Device:C_Small
- added C?: 10p, symbol Device:C_Small
- added C? (x4): 10u, Capacitor_SMD:C_0603_1608Metric_Pad1.05x0.95mm_HandSolder, symbol Device:C_Small
- added D?: LED_Charge, LED_SMD:LED_0603_1608Metric_Pad1.05x0.95mm_HandSolder, symbol Device:LED_Small
- added J?: Conn_I2C, Connector_PinHeader_2.54mm:PinHeader_1x04_P2.54mm_Vertical, symbol Connector_Generic:Conn_01x04
- added J?: Conn_01x03, symbol Connector_Generic:Conn_01x03
- added L? (x2): 2.2u, micelib:SPM3015-xRxM-LR, symbol Device:L_Small
- added R?: 10m, micelib:C_0402_1005Metric_HandSoldering, symbol Device:R_Small
- added R?: 1k, micelib:C_0402_1005Metric_HandSoldering, symbol Device:R_Small
- added U?: INA219AIDCNR, Package_TO_SOT_SMD:SOT-23-8_Handsoldering, symbol dk_PMIC-Current-Regulation-Management:INA219AIDCNR
- added U?: MPU-9250, Sensor_Motion:InvenSense_QFN-24_3x3mm_P0.4mm, symbol Sensor_Motion:MPU-9250
- added U? (x2): TPS63001, micelib:WSON-10-1EP_2x3mm_P0.5mm_EP0.84x2.4mm_TPS6300x, symbol micelib:TPS6300x
- C3: value 10u -> 100u; footprint Capacitor_SMD:C_0603_1608Metric_Pad1.05x0.95mm_HandSolder -> (none)
Connections:
- net labels added: +3.3VA, IMU_CS
- net labels removed: -BATT, OC, OD, PWM1
- wire segments 482 -> 532
- no-connect marks 21 -> 23
Other:
- note added: "Charge"
- note added: "I2C"
- note added: "IMU"
- note added: "LiPo"
- note removed: "Charge\n\nController"
- note removed: "LiPo\n&\nProtection"
- note removed: "Light"
- note removed: "Selector"
- moved on the sheet: BT1, C1, C10, C12, C13, C15, C3, C4, C6, C7, C8, C9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

Commit message: add new schematic
Parts:
- added C10: 10u, micelib:C_0402_1005Metric_HandSoldering, symbol Device:C_Small
- added C11, C14: 0.1u, micelib:C_0402_1005Metric_HandSoldering, symbol Device:C_Small
- added D1: SS2040FL, Diode_SMD:D_SOD-123F, symbol Device:D_Schottky_Small
- C26: renamed from C16; value 10u -> 22u
- gave numbers to parts that had none: 21
- renumbered C7 to C13, C10 to C15, C8 to C2, C15 to C20, C14 to C23, C12 to C24, C13 to C25, C17 to C27, C9 to C4, C4 to C7, C6 to C9, D9 to D10, D1 to D3, D3 to D5, D5 to D6, D6 to D7, D7 to D8, D4 to D9, J1 to J2, J5 to J6, J6 to J7, Q3 to Q1, Q1 to Q2, Q2 to Q3, Q9 to Q7, Q7 to Q8, Q8 to Q9, R10 to R1, R13 to R10, R16 to R11, R14 to R12, R15 to R13, R17 to R15, R19 to R16, R20 to R18, R22 to R19, R1 to R2, R21 to R20, R18 to R21, R23 to R22, R25 to R23, R28 to R24, R36 to R25, R30 to R26, R29 to R27, R26 to R28, R31 to R29, R2 to R3, R27 to R30, R32 to R31, R37 to R32, R3 to R4, R8 to R7, R11 to R8, R12 to R9, U4 to U5, U7 to U8
Connections:
- net +3.3VA: now also D6.1 (+VCC), C10.1
- net +3V3: now also C6.2, U2.13 (VDD), U2.8 (VDDIO); no longer C6.1, D6.1 (+VCC)
- net EN: now also C11.1
- net GNDD: now also C5.2, C6.1, C8.2, SW1.2, U2.18 (GND), U2.20 (RESV_GND), C10.2, C11.2, C14.2
- net IO0: now also C14.1
- net VBUS: now also D1.1 (K); no longer J2.1 (VBUS)
- net at Q3.1 (B): now also R6.1
- new net: D1.2 (A), J2.1 (VBUS)
Other:
- moved on the sheet: BT1, C13, C15, C5, C6, R3, R4, R6, SW1, SW2

Commit message: ToDo : IMU Range Settings
Parts:
- removed R8: 47, micelib:C_0402_1005Metric_HandSoldering, symbol Device:R_Small
- added J10, J11, J12, J13, J9: Conn_01x01, Connector_PinHeader_2.00mm:PinHeader_1x01_P2.00mm_Vertical, symbol Connector_Generic:Conn_01x01
- added J14, J15: Conn_01x02, Connector_PinHeader_2.00mm:PinHeader_1x02_P2.00mm_Vertical, symbol Connector_Generic:Conn_01x02
- added J8: Conn_01x05, Connector_PinHeader_2.54mm:PinHeader_1x05_P2.54mm_Vertical, symbol Connector_Generic:Conn_01x05
- C3: footprint (none) -> Capacitor_SMD:C_1210_3225Metric_Pad1.42x2.65mm_HandSolder
- C5, C6, C8: footprint (none) -> micelib:C_0402_1005Metric_HandSoldering
- J1: footprint (none) -> Connector_PinHeader_2.54mm:PinHeader_1x03_P2.54mm_Vertical
- R17: footprint micelib:C_0402_1005Metric_HandSoldering -> Resistor_SMD:R_1206_3216Metric_Pad1.42x1.75mm_HandSolder
- U2: footprint Sensor_Motion:InvenSense_QFN-24_3x3mm_P0.4mm -> micelib:InvenSense_QFN-24_3x3mm_P0.4mm_HandSoldering
Connections:
- net +3.3VA: now also J8.1 (Pin_1), J9.1 (Pin_1); no longer R24.2, R26.1, R29.1
- net +3V3: now also R24.2, R26.1, R29.1, J13.1 (Pin_1), J8.5 (Pin_5)
- net +5V: now also J11.1 (Pin_1), J8.3 (Pin_3); no longer J4.2 (Pin_2)
- net ADC1_Batt: now also J12.1 (Pin_1), J8.4 (Pin_4)
- net D+: now also J14.1 (Pin_1), J15.1 (Pin_1)
- net D-: now also J14.2 (Pin_2), J15.2 (Pin_2)
- net GNDD: now also J10.1 (Pin_1), J8.2 (Pin_2)
- net at Q5.1 (G), R10.2: now also SW3.2 (B), SW3.3 (C)
- no-connect marks 23 -> 24
Other:
- moved on the sheet: C5, C6, C8, U2
