File: schematic/schematic/schematic.kicad_pcb (KiCad board)
At the start: 2 copper layers, 32.4 x 43.4 mm, 117 parts, among them J1 USB_A, J10 Conn_Tale, J2 USB_B_Micro, J3 Conn_PWM0, J4 Conn_PWM1, J5 Conn_SPI, J6 Conn_I2C, J7 Conn_GPIO, J8 Conn_Tale, J9 Conn_M5StickV, M1 Motor_DC, Q1 SS8050, Q2 SS8050, Q3 IRLML6402, Q4 PJE260N02, Q5 IRLML6402, Q6 PJE260N02, Q7 PJE260N02, SW1 SW_EN, SW2 SW_IO0, SW3 PS-85N, U1 TPS63002, U10 MPU-9250, U11 MPU-9250, U2 TPS63001, U3 MCP73831-5-OT, U4 FT231XS, U5 DW01-P, U6 BR8205, U7 TB6612FNG, U8 ESP32-WROOM-32D

Commit message: 配置開始
Parts:
- added J11: Conn_01x07, Connector_PinSocket_2.54mm:PinSocket_1x07_P2.54mm_Vertical, F.Cu at (122.8, 52.7)
- added J12: Conn_01x07, Connector_PinSocket_2.54mm:PinSocket_1x07_P2.54mm_Vertical, B.Cu at (117.8, 52.7)
- added J13: Conn_01x04, Connector_PinSocket_2.54mm:PinSocket_1x04_P2.54mm_Vertical, F.Cu at (202.5, 113.3)
- added J14: Conn_01x04, Connector_PinSocket_2.54mm:PinSocket_1x04_P2.54mm_Vertical, F.Cu at (206.1, 113.3)
- U10: moved to B.Cu
- U4, U7: moved to F.Cu
- moved SW2 98.7 mm to (169.8, 124.6)
- moved U4 81.5 mm to (162.7, 130.0), turned to 0 degrees
- moved R24 80.4 mm to (185.0, 126.8)
- moved U7 75.6 mm to (154.5, 129.8), turned to 0 degrees
- moved J2 75.5 mm to (141.8, 145.2)
- moved J1 75.3 mm to (129.2, 144.8)
- moved C8 73.9 mm to (181.3, 131.4)
- moved U8 73.7 mm to (136.8, 72.3), turned to 90 degrees
- moved U10 68.9 mm to (142.3, 54.6), turned to 180 degrees
- moved U11 67.4 mm to (140.3, 90.1), turned to 180 degrees
- moved C9 66.7 mm to (176.6, 134.0)
- moved D2 65.4 mm to (188.7, 113.9)
- moved C12 64.2 mm to (178.5, 129.4)
- moved C10 61.8 mm to (174.1, 137.8)
- moved BT1 58.5 mm to (90.1, 91.1), turned to 90 degrees
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Connections:
- C11 pad 1: GND -> GNDD
- C12 pad 2: GND -> GNDD
- C5 pad 1: GND -> GNDD
- C8 pad 2: GND -> GNDD
- J3 pad 3: GND -> GNDD
- J4 pad 3: GND -> GNDD
Other:
- board size 32.4 x 43.4 mm -> 60.8 x 47.4 mm

Commit message: Pin Assign test
Parts:
- removed J10, J8: Conn_Tale, Connector_PinHeader_2.54mm:PinHeader_1x05_P2.54mm_Vertical
- added R29: 10k, micelib:C_0402_1005Metric_HandSoldering, F.Cu at (125.0, 47.1)
- added U9: INA219AIDCNR, Package_TO_SOT_SMD:SOT-23-8_Handsoldering, F.Cu at (194.8, 114.8)
- BT1, J11, U8: moved to B.Cu
- J12: moved to F.Cu
- U1: footprint Connector_PinHeader_2.54mm:PinHeader_1x05_P2.54mm_Vertical -> micelib:WSON-10-1EP_2x3mm_P0.5mm_EP0.84x2.4mm_TPS6300x
- moved BT1 2.12 mm to (90.9, 89.1), turned to 270 degrees
- turned U10 to 90 degrees
- turned J11 to 270 degrees
- turned J12 to 270 degrees
- turned U8 to 270 degrees

Commit message: 地獄の配線
Parts:
- removed C14, C26, C8: 0.1u, micelib:C_0402_1005Metric_HandSoldering
- removed C16: 4.7u, micelib:C_0402_1005Metric_HandSoldering
- removed C4, C5: 10u, Capacitor_SMD:C_0603_1608Metric_Pad1.05x0.95mm_HandSolder
- removed D1: SS2040FL, Diode_SMD:D_SOD-123F
- removed J13, J14: Conn_01x04, Connector_PinSocket_2.54mm:PinSocket_1x04_P2.54mm_Vertical
- removed J5: Conn_SPI, Connector_PinHeader_2.54mm:PinHeader_1x05_P2.54mm_Vertical
- removed J7: Conn_GPIO, Connector_PinHeader_2.54mm:PinHeader_1x02_P2.54mm_Vertical
- removed JP2: Jumper, Jumper:SolderJumper-2_P1.3mm_Bridged2Bar_Pad1.0x1.5mm
- removed TP1: 5V, Connector_PinHeader_1.27mm:PinHeader_1x01_P1.27mm_Vertical
- removed TP2: 3.3V, Connector_PinHeader_1.27mm:PinHeader_1x01_P1.27mm_Vertical
- removed TP3: +VBAT, Connector_PinHeader_1.27mm:PinHeader_1x01_P1.27mm_Vertical
- added J10: Conn_Tale, Connector_PinHeader_2.54mm:PinHeader_1x05_P2.54mm_Vertical, F.Cu at (128.8, 96.8)
- added J8: Conn_Tale, Connector_PinHeader_2.54mm:PinHeader_1x05_P2.54mm_Vertical, B.Cu at (126.6, 91.7)
- BT1, U10: moved to F.Cu
- C13, C17, C19, C20, C22, C25, D7, J2, J6, J9, L1, L2, Q4, Q7, R10, R16, R17, R18, R2, R22, R23, R24, R33, R7, R9, SW1, SW2, TP4, TP5, U3, U5, U7: moved to B.Cu
- J1: value USB_A -> Conn_01x05; footprint micelib:USB_A_Vertical -> Connector_PinHeader_1.00mm:PinHeader_2x03_P1.00mm_Vertical_SMD; moved to B.Cu
- J11, J12: footprint Connector_PinSocket_2.54mm:PinSocket_1x07_P2.54mm_Vertical -> Connector_PinHeader_1.00mm:PinHeader_2x04_P1.00mm_Vertical_SMD
- J3: value Conn_PWM0 -> Conn_02x03_Odd_Even; footprint Connector_PinHeader_2.54mm:PinHeader_1x03_P2.54mm_Vertical -> Connector_PinSocket_2.54mm:PinSocket_2x03_P2.54mm_Vertical
- J4: value Conn_PWM1 -> Conn_01x05; footprint Connector_PinHeader_2.54mm:PinHeader_1x03_P2.54mm_Vertical -> Connector_PinHeader_1.00mm:PinHeader_2x03_P1.00mm_Vertical_SMD
- R15, R21: value 100k -> 10k
- R20: value 100k -> 10k; moved to B.Cu
- SW3: value PS-85N -> SW_SPDT; footprint micelib:PS-85 -> Connector_PinSocket_2.54mm:PinSocket_1x03_P2.54mm_Vertical
- U8: footprint RF_Module:ESP32-WROOM-32 -> micelib:ESP32-WROOM-32_Hand
- moved R27 128.0 mm to (102.5, 54.7), turned to 270 degrees
- moved C22 126.3 mm to (103.0, 53.9)
- moved R28 124.7 mm to (103.8, 54.7), turned to 270 degrees
- moved R11 123.2 mm to (103.2, 56.5), turned to 180 degrees
- moved R9 115.9 mm to (92.1, 54.6), turned to 180 degrees
- moved R17 113.9 mm to (96.7, 53.6)
- moved SW3 107.6 mm to (88.9, 57.2), turned to 180 degrees
- moved U9 107.0 mm to (107.5, 53.0)
- moved D6 104.2 mm to (96.9, 55.3)
- moved TP6 99.9 mm to (95.7, 70.5)
- moved M1 99.7 mm to (95.1, 64.6), turned to 180 degrees
- moved R26 96.8 mm to (133.0, 55.4)
- moved C18 96.7 mm to (109.9, 61.0), turned to 90 degrees
- moved C6 94.5 mm to (101.5, 72.5), turned to 90 degrees
- moved C20 94.5 mm to (107.6, 57.6), turned to 90 degrees
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Connections:
- C11 pad 1: GNDD -> +5V
- C11 pad 2: +5V -> GNDD
- C12 pad 1: +5V -> GNDD
- C12 pad 2: GNDD -> +5V
- J1 pad 1: Net-(D1-Pad1) -> GNDD
- J1 pad 2: (no net) -> VBUS
- J1 pad 3: (no net) -> +3V3
- J1 pad 4: GNDD -> +5V
- J1 pad 5: GNDD -> ADC1_Batt
- J11 pad 1: PWM1 -> (no net)
- J11 pad 2: PWM0 -> (no net)
- J12 pad 1: PWM1 -> (no net)
- J12 pad 2: PWM0 -> (no net)
- J3 pad 2: +5V -> PWM1
- J3 pad 3: GNDD -> +5V
- J4 pad 1: PWM1 -> GNDD
- J4 pad 2: +5V -> VBUS
- J4 pad 3: GNDD -> +3V3
- J9 pad 2: (no net) -> +5V
- SW3 pad 2: GND -> Net-(R9-Pad2)
- SW3 pad 3: GND -> Net-(R9-Pad2)
- U8 pad 6: GPIO34 -> ADC1_Batt
- U8 pad 7: GPIO35 -> (no net)
- U8 pad 9: ADC1_Batt -> (no net)
Routing:
- net +3V3: track 0.00 -> 176.0 mm, vias 0 -> 7
- net +5V: track 0.00 -> 121.7 mm, vias 0 -> 8
- net ADC1_Batt: track 0.00 -> 69.0 mm, vias 0 -> 7
- net I2C_SCL: track 0.00 -> 65.2 mm, vias 0 -> 7
- net MD_IN2: track 0.00 -> 60.0 mm, vias 0 -> 5
- net I2C_SDA: track 0.00 -> 53.9 mm, vias 0 -> 6
- net PWM_MD: track 0.00 -> 48.9 mm, vias 0 -> 7
- net LED_LEFT: track 0.00 -> 45.1 mm, vias 0 -> 6
- net -BATT: track 0.00 -> 45.0 mm, vias 0 -> 2
- net MD_IN1: track 0.00 -> 44.6 mm, vias 0 -> 3
- net LED_RIGHT: track 0.00 -> 41.3 mm, vias 0 -> 5
- net DTR: track 0.00 -> 41.0 mm, vias 0 -> 4
- net Net-(Q2-Pad1): track 0.00 -> 40.6 mm, vias 0 -> 2
- net Net-(Q5-Pad1): track 0.00 -> 37.3 mm, vias 0 -> 3
- net VSPI_CLK: track 0.00 -> 36.0 mm, vias 0 -> 4
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Other:
- board size 60.8 x 47.4 mm -> 60.8 x 50.4 mm
- net class +batt added: clearance 0.2, trace_width 1, via_dia 0.8, via_drill 0.4
- net class 3V3: trace_width 0.5 -> 0.75
- net class 5V: trace_width 1.5 -> 0.75
- net class Default: trace_width 0.21 -> 0.18
- rule trace_min: 0.2 -> 0.175
