File: schematic/schematic/schematic.kicad_pcb (KiCad board)
At the start: 2 copper layers, 108 parts, among them IC1 DRV8830, J1 USB_B_Micro, J10 Conn_I2CBridge, J11 Conn_PBridge, J12 Conn__PBridge, J2 Conn_PWM, J3 Conn_GPIO, J4 Conn_M5StickV, J5 Conn_Tale, J6 Conn_Tale, J7 Conn_I2C, J8 Conn_SPI, J9 Conn__I2CBridge, M1 M_Small, Q1 SS8050, Q2 SS8050, Q3 IRLML6402, Q4 PJE260N02, Q5 IRLML6402, Q6 PJE260N02, Q7 BSS138, Q8 BSS138, Q9 PJE260N02, SW1 SW_EN, SW2 SW_IO0, SW3 SW_SPDT, U1 TPS63002, U2 TPS63001, U3 MCP73831-5-OT, U4 FT231XS, U5 DW01-P, U6 BR8205, U7 ESP32-WROOM-32D, U8 INA219AIDCNR

Commit message: やっぱり機能を絞るに限る
Parts:
- removed R34, R35: 10, micelib:C_0402_1005Metric_HandSoldering
- added C21: 0.1u, micelib:C_0402_1005Metric_HandSoldering, B.Cu at (33.4, 64.4)
- C15, C4, C5, C6, D2, D4, D5, IC1, J1, J2, J3, J4, J6, J7, J8, L1, L2, Q3, Q4, Q8, R12, R17, R18, R19, R2, R24, R25, R26, R27, R7, SW1, SW2, U3, U6: moved to B.Cu
- J10: value Conn_I2CBridge -> Conn_01x06
- J12: value Conn__PBridge -> Conn_01x06
- J5: footprint Connector_PinHeader_2.54mm:PinHeader_1x05_P2.54mm_Vertical -> Connector_PinHeader_1.27mm:PinHeader_1x05_P1.27mm_Vertical; moved to B.Cu
- J9: value Conn__I2CBridge -> Conn_01x06
- JP1: value Jumper -> Jumper_NO_Small; footprint Jumper:SolderJumper-2_P1.3mm_Bridged2Bar_Pad1.0x1.5mm -> Jumper:SolderJumper-2_P1.3mm_Open_TrianglePad1.0x1.5mm
- U7: value ESP32-WROOM-32D -> ESP32-WROOM-32D_GND_39; moved to B.Cu
- moved R33 149.7 mm to (29.8, 61.5), turned to 90 degrees
- moved U8 143.7 mm to (36.4, 62.5)
- moved C6 141.1 mm to (27.7, 30.0)
- moved R4 140.7 mm to (29.4, 31.4), turned to 180 degrees
- moved TP1 140.3 mm to (27.1, 31.4)
- moved R3 138.7 mm to (31.6, 35.2), turned to 90 degrees
- moved C19 137.1 mm to (33.0, 61.5), turned to 270 degrees
- moved R2 135.5 mm to (31.5, 32.1), turned to 270 degrees
- moved J12 134.9 mm to (50.6, 32.3), turned to 270 degrees
- moved TP2 133.2 mm to (27.1, 33.5)
- moved BT1 130.9 mm to (23.7, 31.4), turned to 270 degrees
- moved C3 129.5 mm to (42.1, 30.3), turned to 90 degrees
- moved U5 128.6 mm to (34.8, 31.3), turned to 180 degrees
- moved C10 128.4 mm to (30.4, 35.2), turned to 90 degrees
- moved J11 128.4 mm to (55.8, 32.3), turned to 270 degrees
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Connections:
- C1 pad 2: GND -> GNDD
- C16 pad 1: GND -> GNDD
- C17 pad 2: GND -> GNDD
- C19 pad 1: Net-(C19-Pad1) -> +5V
- C19 pad 2: Net-(C19-Pad2) -> MD_VM
- C2 pad 2: GND -> GNDD
- C3 pad 2: GND -> GNDD
- C6 pad 2: GND -> GNDD
- D7 pad 1: Net-(D7-Pad1) -> FAULTn
- D7 pad 2: +5V -> Net-(D7-Pad2)
- D8 pad 1: Net-(D8-Pad1) -> STAT
- D8 pad 2: VBUS -> Net-(D8-Pad2)
- IC1 pad 7: GND -> GNDD
- IC1 pad 8: GND -> GNDD
- J1 pad 5: GND -> GNDD
- J1 pad 6: GND -> GNDD
- J10 pad 3: (no net) -> GNDD
- J10 pad 4: (no net) -> ADC1_Batt
- J10 pad 5: (no net) -> GNDD
- J10 pad 6: (no net) -> GNDD
- J11 pad 5: ADC1_Batt -> GNDD
- J12 pad 2: VBUS -> GNDD
- J12 pad 5: ADC1_Batt -> GNDD
- J12 pad 6: (no net) -> VBUS
- J2 pad 1: PWM0 -> PWM1
- J2 pad 2: PWM1 -> PWM0
- J4 pad 3: ESP32_RX -> ESP32_TX
- J4 pad 4: ESP32_TX -> ESP32_RX
- J5 pad 1: LED_LEFT -> LED_RIGHT
- J5 pad 3: LED_RIGHT -> LED_LEFT
- J6 pad 1: LED_LEFT -> LED_RIGHT
- J6 pad 3: LED_RIGHT -> LED_LEFT
- J7 pad 1: I2C_SCL -> I2C_SDA
- J7 pad 2: I2C_SDA -> I2C_SCL
- J8 pad 1: SPI_CLK -> SPI_MISO
- J8 pad 3: SPI_MISO -> SPI_CLK
- J9 pad 1: I2C_SCL -> GNDD
- J9 pad 2: I2C_SDA -> GNDD
- J9 pad 3: (no net) -> GNDD
- J9 pad 4: (no net) -> ADC1_Batt
- J9 pad 5: (no net) -> I2C_SCL
- J9 pad 6: (no net) -> I2C_SDA
- R1 pad 2: GND -> GNDD
- R10 pad 2: GND -> GNDD
- R20 pad 1: Net-(D7-Pad1) -> +5V
- R20 pad 2: FAULTn -> Net-(D7-Pad2)
- R24 pad 1: Net-(D8-Pad1) -> VBUS
- R24 pad 2: STAT -> Net-(D8-Pad2)
- R7 pad 1: GND -> GNDD
- R9 pad 2: GND -> GNDD
- SW3 pad 1: GND -> GNDD
- U1 pad 11: GND -> GNDD
- U1 pad 3: GND -> GNDD
- U2 pad 11: GND -> GNDD
- U2 pad 3: GND -> GNDD
- U3 pad 2: GND -> GNDD
- U7 pad 39: (no net) -> GNDD
- U8 pad 1: Net-(C19-Pad1) -> +5V
- U8 pad 2: Net-(C19-Pad2) -> MD_VM
Routing:
- net +3V3: track 0.00 -> 202.0 mm, vias 0 -> 14
- net +5V: track 0.00 -> 119.4 mm, vias 0 -> 6
- net ADC1_Batt: track 0.00 -> 94.0 mm, vias 0 -> 7
- net VBUS: track 0.00 -> 59.3 mm, vias 0 -> 6
- net I2C_SDA: track 0.00 -> 53.4 mm, vias 0 -> 3
- net I2C_SCL: track 0.00 -> 43.7 mm, vias 0 -> 5
- net Net-(Q5-Pad1): track 0.00 -> 33.1 mm, vias 0 -> 4
- net +BATT: track 0.00 -> 32.3 mm
- net D-: track 0.00 -> 25.0 mm, vias 0 -> 3
- net VBAT: track 0.00 -> 23.8 mm
- net GNDD: track 0.00 -> 22.9 mm, vias 0 -> 157
- net IO0: track 0.00 -> 21.5 mm, vias 0 -> 4
- net D+: track 0.00 -> 21.2 mm, vias 0 -> 1
- net SPI_MOSI: track 0.00 -> 20.9 mm, vias 0 -> 1
- net GPIO_19: track 0.00 -> 19.0 mm
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- added copper zone on F.Cu, net +3V3
- added copper zone on F.Cu, net +5V
- added copper zone on F.Cu, net GND
- added copper zone on B.Cu, net GNDD
- added copper zone on F.Cu, net GNDD
Other:
- board outline added: 60.8 x 51.4 mm
- net class Default: trace_width 0.25 -> 0.18
- net class Motor added: clearance 0.2, trace_width 0.75, via_dia 0.8, via_drill 0.4
- net class Power added: clearance 0.2, trace_width 0.4, via_dia 0.8, via_drill 0.4
- rule trace_min: 0.2 -> 0.175
- board text added: "CBUS1"
- board text added: "CBUS2"
- board text added: "P0"
- board text added: "P1+-"

Commit message: ビアをいっぱい打ち込んだ
Routing:
- net +3V3: track 202.0 -> 203.7 mm
- net +BATT: track 32.3 -> 33.3 mm
- net GNDD: vias 157 -> 183
Other:
- board text added: "5 18 19"
- board text added: "SDA SCL 3.3V -"

Commit message: とりあえずのデータは完成
Parts:
- added G***: LOGO, micelib:icon_mini, F.Cu at (46.7, 59.1)
- added REF**: PinHeader_1x01_P1.27mm_Vertical, Connector_PinHeader_1.27mm:PinHeader_1x01_P1.27mm_Vertical, F.Cu at (80.0, 40.0)
- added REF**: PinHeader_1x01_P1.27mm_Vertical, Connector_PinHeader_1.27mm:PinHeader_1x01_P1.27mm_Vertical, F.Cu at (26.4, 40.0)
Routing:
- net SPI_MOSI: track 20.9 -> 18.8 mm
