File: schematic/schematic/Sensors.sch (KiCad schematic (older format))
At the start: 13 parts, among them U10 MPU-9250, U11 MPU-9250, U9 INA219AIDCNR

Commit message: assign footprint
Parts:
- C22, C29, C30, C32, C33: footprint (none) -> micelib:C_0402_1005Metric_HandSoldering
- C28, C31: footprint (none) -> micelib:C_0201_0603Metric_HandSoldering
Changed lines of the file:
@@
 F 0 "C22" H 1550 1350 50  0000 L CNN
 F 1 "0.1u" H 1550 1250 50  0000 L CNN
-F 2 "" H 1450 1300 50  0001 C CNN
+F 2 "micelib:C_0402_1005Metric_HandSoldering" H 1450 1300 50  0001 C CNN
 F 3 "~" H 1450 1300 50  0001 C CNN
 	1    1450 1300
@@
 F 0 "C30" V 3471 4500 50  0000 C CNN
 F 1 "0.1u" V 3562 4500 50  0000 C CNN
-F 2 "" H 3700 4500 50  0001 C CNN
+F 2 "micelib:C_0402_1005Metric_HandSoldering" H 3700 4500 50  0001 C CNN
 F 3 "~" H 3700 4500 50  0001 C CNN
 	1    3700 4500
@@
 F 0 "C33" V 6271 4500 50  0000 C CNN
 F 1 "0.1u" V 6362 4500 50  0000 C CNN
-F 2 "" H 6500 4500 50  0001 C CNN
+F 2 "micelib:C_0402_1005Metric_HandSoldering" H 6500 4500 50  0001 C CNN
 F 3 "~" H 6500 4500 50  0001 C CNN
 	1    6500 4500
@@
 F 0 "C28" H 1742 3496 50  0000 L CNN
 F 1 "10n" H 1742 3405 50  0000 L CNN
-F 2 "" H 1650 3450 50  0001 C CNN
+F 2 "micelib:C_0201_0603Metric_HandSoldering" H 1650 3450 50  0001 C CNN
 F 3 "~" H 1650 3450 50  0001 C CNN
 	1    1650 3450
@@
 F 0 "C29" H 2092 3496 50  0000 L CNN
 F 1 "0.1u" H 2092 3405 50  0000 L CNN
-F 2 "" H 2000 3450 50  0001 C CNN
+F 2 "micelib:C_0402_1005Metric_HandSoldering" H 2000 3450 50  0001 C CNN
 F 3 "~" H 2000 3450 50  0001 C CNN
 	1    2000 3450
@@
 F 0 "C31" H 4542 3496 50  0000 L CNN
 F 1 "10n" H 4542 3405 50  0000 L CNN
-F 2 "" H 4450 3450 50  0001 C CNN
+F 2 "micelib:C_0201_0603Metric_HandSoldering" H 4450 3450 50  0001 C CNN
 F 3 "~" H 4450 3450 50  0001 C CNN
 	1    4450 3450
@@
 F 0 "C32" H 4892 3496 50  0000 L CNN
 F 1 "0.1u" H 4892 3405 50  0000 L CNN
-F 2 "" H 4800 3450 50  0001 C CNN
+F 2 "micelib:C_0402_1005Metric_HandSoldering" H 4800 3450 50  0001 C CNN
 F 3 "~" H 4800 3450 50  0001 C CNN
 	1    4800 3450

Commit message: wip: add another layer
Parts:
- R11, R27, R28: footprint (none) -> micelib:C_0402_1005Metric_HandSoldering
- U10, U11: footprint Sensor_Motion:InvenSense_QFN-24_3x3mm_P0.4mm -> micelib:InvenSense_QFN-24_3x3mm_P0.4mm_HandSoldering
Changed lines of the file:
@@
 F 0 "R27" V 1200 1150 50  0000 C CNN
 F 1 "10" V 1400 1150 50  0000 C CNN
-F 2 "" H 1300 1150 50  0001 C CNN
+F 2 "micelib:C_0402_1005Metric_HandSoldering" H 1300 1150 50  0001 C CNN
 F 3 "~" H 1300 1150 50  0001 C CNN
 	1    1300 1150
@@
 F 0 "R28" V 1200 1450 50  0000 C CNN
 F 1 "10" V 1400 1450 50  0000 C CNN
-F 2 "" H 1300 1450 50  0001 C CNN
+F 2 "micelib:C_0402_1005Metric_HandSoldering" H 1300 1450 50  0001 C CNN
 F 3 "~" H 1300 1450 50  0001 C CNN
 	1    1300 1450
@@
 F 0 "R11" H 1300 1250 50  0000 C CNN
 F 1 "2m" H 1250 1350 50  0000 C CNN
-F 2 "" H 1150 1300 50  0001 C CNN
+F 2 "micelib:C_0402_1005Metric_HandSoldering" H 1150 1300 50  0001 C CNN
 F 3 "~" H 1150 1300 50  0001 C CNN
 	1    1150 1300
@@
 F 0 "U10" H 2850 4300 50  0000 C CNN
 F 1 "MPU-9250" H 2850 4200 50  0000 C CNN
-F 2 "Sensor_Motion:InvenSense_QFN-24_3x3mm_P0.4mm" H 2850 3300 50  0001 C CNN
+F 2 "micelib:InvenSense_QFN-24_3x3mm_P0.4mm_HandSoldering" H 2850 3300 50  0001 C CNN
 F 3 "https://store.invensense.com/datasheets/invensense/MPU9250REV1.0.pdf" H 2850 4150 50  0001 C CNN
 	1    2850 4300
@@
 F 0 "U11" H 5650 4300 50  0000 C CNN
 F 1 "MPU-9250" H 5650 4200 50  0000 C CNN
-F 2 "Sensor_Motion:InvenSense_QFN-24_3x3mm_P0.4mm" H 5650 3300 50  0001 C CNN
+F 2 "micelib:InvenSense_QFN-24_3x3mm_P0.4mm_HandSoldering" H 5650 3300 50  0001 C CNN
 F 3 "https://store.invensense.com/datasheets/invensense/MPU9250REV1.0.pdf" H 5650 4150 50  0001 C CNN
 	1    5650 4300

Commit message: 配置開始
Parts:
- added J11, J12: Conn_01x07, Connector_PinSocket_2.54mm:PinSocket_1x07_P2.54mm_Vertical, symbol Connector_Generic:Conn_01x07
- added J13, J14: Conn_01x04, Connector_PinSocket_2.54mm:PinSocket_1x04_P2.54mm_Vertical, symbol Connector_Generic:Conn_01x04
Connections:
- net +3V3: now also J13.2 (Pin_2), J14.2 (Pin_2)
- net +5V: now also J13.3 (Pin_3), J14.3 (Pin_3)
- net I2C_SCL: now also J11.3 (Pin_3), J12.3 (Pin_3)
- net I2C_SDA: now also J11.4 (Pin_4), J12.4 (Pin_4)
- new net ADC1_Batt: J13.4 (Pin_4), J14.4 (Pin_4)
- new net GND: J13.1 (Pin_1), J14.1 (Pin_1)
- new net MD_IN1: J11.6 (Pin_6), J12.6 (Pin_6)
- new net MD_IN2: J11.5 (Pin_5), J12.5 (Pin_5)
- new net PWM0: J11.2 (Pin_2), J12.2 (Pin_2)
- new net PWM1: J11.1 (Pin_1), J12.1 (Pin_1)
- new net PWM_MD: J11.7 (Pin_7), J12.7 (Pin_7)
Changed lines of the file:
@@
 Wire Notes Line
 	6800 6450 600  6450
+Text GLabel 3500 700  2    50   Input ~ 0
+PWM_MD
+Text GLabel 3500 800  2    50   Input ~ 0
+MD_IN1
+Text GLabel 3500 900  2    50   Input ~ 0
+MD_IN2
+Text GLabel 3500 1000 2    50   Input ~ 0
+I2C_SDA
+Text GLabel 3500 1100 2    50   Input ~ 0
+I2C_SCL
+$Comp
+L power:GND #PWR?
+U 1 1 5EC61195
+P 4650 1950
+AR Path="/5EC61195" Ref="#PWR?"  Part="1"
+AR Path="/5E247314/5EC61195" Ref="#PWR075"  Part="1"
+F 0 "#PWR075" H 4650 1700 50  0001 C CNN
+F 1 "GND" H 4650 1800 50  0000 C CNN
+F 2 "" H 4650 1950 50  0001 C CNN
+F 3 "" H 4650 1950 50  0001 C CNN
+	1    4650 1950
+	1    0    0    -1
+$EndComp
+Text GLabel 4850 1600 2    50   Input ~ 0
+ADC1_Batt
+Wire Wire Line
+	4650 1950 4650 1900
+$Comp
+L Connector_Generic:Conn_01x04 J14
+U 1 1 5ECB2FF3
+P 4300 1800
+F 0 "J14" H 4220 1375 50  0000 C CNN
+F 1 "Conn_01x04" H 4220 1466 50  0000 C CNN
+F 2 "Connector_PinSocket_2.54mm:PinSocket_1x04_P2.54mm_Vertical" H 4300 1800 50  0001 C CNN
+F 3 "~" H 4300 1800 50  0001 C CNN
+	1    4300 1800
+	-1   0    0    1
+$EndComp
+$Comp
+L Connector_Generic:Conn_01x04 J13
+U 1 1 5ECB3055
+P 4300 1150
+F 0 "J13" H 4220 725 50  0000 C CNN
+F 1 "Conn_01x04" H 4220 816 50  0000 C CNN
+F 2 "Connector_PinSocket_2.54mm:PinSocket_1x04_P2.54mm_Vertical" H 4300 1150 50  0001 C CNN
+F 3 "~" H 4300 1150 50  0001 C CNN
+	1    4300 1150
+	-1   0    0    1
+$EndComp
+Wire Wire Line
+	4500 1900 4650 1900
+$Comp
+L power:+3V3 #PWR077
+U 1 1 5ECBE3B6
+P 5550 1550
+F 0 "#PWR077" H 5550 1400 50  0001 C CNN
+F 1 "+3V3" H 5565 1723 50  0000 C CNN
+F 2 "" H 5550 1550 50  0001 C CNN
+F 3 "" H 5550 1550 50  0001 C CNN
+	1    5550 1550
+	1    0    0    -1
+$EndComp
+$Comp
+L power:+5V #PWR076
+U 1 1 5ECBE416
+P 5350 1550
+F 0 "#PWR076" H 5350 1400 50  0001 C CNN
+F 1 "+5V" H 5365 1723 50  0000 C CNN
+F 2 "" H 5350 1550 50  0001 C CNN
+F 3 "" H 5350 1550 50  0001 C CNN
+	1    5350 1550
+	1    0    0    -1
+$EndComp
+Wire Wire Line
+	5350 1550 5350 1700
+Wire Wire Line
+	4650 1900 4650 1250
+Wire Wire Line
+	4650 1250 4500 1250
+Connection ~ 4650 1900
+Wire Wire Line
+	4500 1700 4750 1700
+Wire Wire Line
+	4500 1800 4700 1800
+Wire Wire Line
+	4500 1150 4700 1150
+Wire Wire Line
+	4700 1150 4700 1800
+Connection ~ 4700 1800
+Wire Wire Line
+	4500 1050 4750 1050
+Wire Wire Line
+	4750 1050 4750 1700
+Connection ~ 4750 1700
+Wire Wire Line
+	5550 1550 5550 1800
+Wire Wire Line
+	4750 1700 5350 1700
+Wire Wire Line
+	4700 1800 5550 1800
+Wire Wire Line
+	4500 950  4800 950
+Wire Wire Line
+	4800 950  4800 1600
+Wire Wire Line
+	4800 1600 4500 1600
+Wire Wire Line
+	4850 1600 4800 1600
+Connection ~ 4800 1600
+Text GLabel 3500 1200 2    50   Input ~ 0
+PWM0
+Text GLabel 3500 1300 2    50   Input ~ 0
+PWM1
+$Comp
+L Connector_Generic:Conn_01x07 J11
+U 1 1 5ED4250E
+P 2800 1000
+F 0 "J11" H 2700 550 50  0000 C CNN
+F 1 "Conn_01x07" H 2700 600 50  0000 C CNN
+F 2 "Connector_PinSocket_2.54mm:PinSocket_1x07_P2.54mm_Vertical" H 2800 1000 50  0001 C CNN
+F 3 "~" H 2800 1000 50  0001 C CNN
+	1    2800 1000
+	-1   0    0    1
+$EndComp
+$Comp
+L Connector_Generic:Conn_01x07 J12
+U 1 1 5ED425C0
+P 2800 1900
+F 0 "J12" H 2700 1450 50  0000 C CNN
+F 1 "Conn_01x07" H 2700 1500 50  0000 C CNN
+F 2 "Connector_PinSocket_2.54mm:PinSocket_1x07_P2.54mm_Vertical" H 2800 1900 50  0001 C CNN
+F 3 "~" H 2800 1900 50  0001 C CNN
+	1    2800 1900
+	-1   0    0    1
+$EndComp
+Wire Wire Line
+	3000 700  3150 700
+Wire Wire Line
+	3000 800  3200 800
+Wire Wire Line
+	3000 900  3250 900
+Wire Wire Line
+	3000 1000 3300 1000
+Wire Wire Line
+	3000 1100 3350 1100
+Wire Wire Line
+	3000 1200 3400 1200
+Wire Wire Line
+	3000 1600 3150 1600
+Wire Wire Line
+	3150 1600 3150 700
+Connection ~ 3150 700
+Wire Wire Line
+	3200 1700 3000 1700
+Wire Wire Line
+	3000 1800 3250 1800
+Wire Wire Line
+	3250 1800 3250 900
+Connection ~ 3250 900
+Wire Wire Line
+	3200 1700 3200 800
+Connection ~ 3200 800
+Wire Wire Line
+	3300 1000 3300 1900
+Wire Wire Line
+	3300 1900 3000 1900
+Connection ~ 3300 1000
+Wire Wire Line
+	3000 2000 3350 2000
+Wire Wire Line
+	3350 2000 3350 1100
+Connection ~ 3350 1100
+Wire Wire Line
+	3400 1200 3400 2100
+Wire Wire Line
+	3400 2100 3000 2100
+Connection ~ 3400 1200
+Wire Wire Line
+	3000 1300 3450 1300
+Wire Wire Line
+	3400 1200 3500 1200
+Wire Wire Line
+	3350 1100 3500 1100
+Wire Wire Line
+	3300 1000 3500 1000
+Wire Wire Line
+	3250 900  3500 900
+Wire Wire Line
+	3200 800  3500 800
+Wire Wire Line
+	3150 700  3500 700
+Wire Wire Line
+	3450 1300 3450 2200
+Wire Wire Line
+	3450 2200 3000 2200
 Wire Bus Line
 	1550 5550 1550 5950
@@
 Wire Bus Line
 	4000 3100 4000 4100
+Connection ~ 3450 1300
+Wire Wire Line
+	3450 1300 3500 1300
 $EndSCHEMATC

Commit message: Pin Assign test
Parts:
- added R29: 10k, micelib:C_0402_1005Metric_HandSoldering, symbol Device:R_Small
- U9: footprint digikey-footprints:SOT-23-8 -> Package_TO_SOT_SMD:SOT-23-8_Handsoldering
Connections:
- net GNDD: now also R29.2
- net VSPI_CS1: now also R29.1
Changed lines of the file:
@@
 F 0 "U9" H 2150 1550 60  0000 L CNN
 F 1 "INA219AIDCNR" V 2350 1200 60  0000 L CNN
-F 2 "digikey-footprints:SOT-23-8" H 2400 1750 60  0001 L CNN
+F 2 "Package_TO_SOT_SMD:SOT-23-8_Handsoldering" H 2400 1750 60  0001 L CNN
 F 3 "http://www.ti.com/lit/ds/symlink/ina219.pdf" H 2400 1850 60  0001 L CNN
 F 4 "296-23770-1-ND" H 2400 1950 60  0001 L CNN "Digi-Key_PN"
@@
 CS1
 Wire Wire Line
-	1100 6050 1450 6050
+	1100 6050 1400 6050
 Wire Wire Line
 	1100 5950 1450 5950
@@
 Wire Wire Line
 	3450 2200 3000 2200
+Connection ~ 3450 1300
+Wire Wire Line
+	3450 1300 3500 1300
+$Comp
+L Device:R_Small R29
+U 1 1 5E22EBA7
+P 1400 6200
+F 0 "R29" H 1459 6246 50  0000 L CNN
+F 1 "10k" H 1459 6155 50  0000 L CNN
+F 2 "micelib:C_0402_1005Metric_HandSoldering" H 1400 6200 50  0001 C CNN
+F 3 "~" H 1400 6200 50  0001 C CNN
+	1    1400 6200
+	1    0    0    -1
+$EndComp
+Wire Wire Line
+	1400 6100 1400 6050
+Connection ~ 1400 6050
+Wire Wire Line
+	1400 6050 1450 6050
+Wire Wire Line
+	1400 6300 1400 6350
+$Comp
+L power:GNDD #PWR078
+U 1 1 5E236C74
+P 1400 6350
+F 0 "#PWR078" H 1400 6100 50  0001 C CNN
+F 1 "GNDD" H 1600 6300 50  0000 C CNN
+F 2 "" H 1400 6350 50  0001 C CNN
+F 3 "" H 1400 6350 50  0001 C CNN
+	1    1400 6350
+	1    0    0    -1
+$EndComp
 Wire Bus Line
 	1550 5550 1550 5950
@@
 Wire Bus Line
 	4000 3100 4000 4100
-Connection ~ 3450 1300
-Wire Wire Line
-	3450 1300 3500 1300
 $EndSCHEMATC

Commit message: 地獄の配線
Parts:
- removed J13, J14: Conn_01x04, Connector_PinSocket_2.54mm:PinSocket_1x04_P2.54mm_Vertical, symbol Connector_Generic:Conn_01x04
- added J1, J4: Conn_01x05, Connector_PinHeader_1.00mm:PinHeader_2x03_P1.00mm_Vertical_SMD, symbol Connector_Generic:Conn_01x05
- J11, J12: footprint Connector_PinSocket_2.54mm:PinSocket_1x07_P2.54mm_Vertical -> Connector_PinHeader_1.00mm:PinHeader_2x04_P1.00mm_Vertical_SMD
Connections:
- net +3V3: now also J1.3 (Pin_3), J4.3 (Pin_3)
- net +5V: now also J1.4 (Pin_4), J4.4 (Pin_4)
- net ADC1_Batt: now also J1.5 (Pin_5), J4.5 (Pin_5)
- net GNDD: now also J1.1 (Pin_1), J4.1 (Pin_1)
- net PWM0: no longer names the net of J11.2 (Pin_2)
- net PWM0: no longer J12.2 (Pin_2)
- net PWM1: no longer names the net of J11.1 (Pin_1)
- net PWM1: no longer J12.1 (Pin_1)
- new net VBUS: J1.2 (Pin_2), J4.2 (Pin_2)
- no-connect marks 10 -> 14
Changed lines of the file:
@@
 Text GLabel 3500 1100 2    50   Input ~ 0
 I2C_SCL
-$Comp
-L power:GND #PWR?
-U 1 1 5EC61195
-P 4650 1950
-AR Path="/5EC61195" Ref="#PWR?"  Part="1"
-AR Path="/5E247314/5EC61195" Ref="#PWR075"  Part="1"
-F 0 "#PWR075" H 4650 1700 50  0001 C CNN
-F 1 "GND" H 4650 1800 50  0000 C CNN
-F 2 "" H 4650 1950 50  0001 C CNN
-F 3 "" H 4650 1950 50  0001 C CNN
-	1    4650 1950
-	1    0    0    -1
-$EndComp
 Text GLabel 4850 1600 2    50   Input ~ 0
 ADC1_Batt
 Wire Wire Line
-	4650 1950 4650 1900
-$Comp
-L Connector_Generic:Conn_01x04 J14
-U 1 1 5ECB2FF3
-P 4300 1800
-F 0 "J14" H 4220 1375 50  0000 C CNN
-F 1 "Conn_01x04" H 4220 1466 50  0000 C CNN
-F 2 "Connector_PinSocket_2.54mm:PinSocket_1x04_P2.54mm_Vertical" H 4300 1800 50  0001 C CNN
-F 3 "~" H 4300 1800 50  0001 C CNN
-	1    4300 1800
-	-1   0    0    1
-$EndComp
-$Comp
-L Connector_Generic:Conn_01x04 J13
-U 1 1 5ECB3055
-P 4300 1150
-F 0 "J13" H 4220 725 50  0000 C CNN
-F 1 "Conn_01x04" H 4220 816 50  0000 C CNN
-F 2 "Connector_PinSocket_2.54mm:PinSocket_1x04_P2.54mm_Vertical" H 4300 1150 50  0001 C CNN
-F 3 "~" H 4300 1150 50  0001 C CNN
-	1    4300 1150
-	-1   0    0    1
-$EndComp
-Wire Wire Line
-	4500 1900 4650 1900
+	4650 2050 4650 2000
 $Comp
 L power:+3V3 #PWR077
@@
 	5350 1550 5350 1700
 Wire Wire Line
-	4650 1900 4650 1250
-Wire Wire Line
-	4650 1250 4500 1250
-Connection ~ 4650 1900
-Wire Wire Line
-	4500 1700 4750 1700
-Wire Wire Line
-	4500 1800 4700 1800
-Wire Wire Line
-	4500 1150 4700 1150
-Wire Wire Line
-	4700 1150 4700 1800
-Connection ~ 4700 1800
-Wire Wire Line
-	4500 1050 4750 1050
-Wire Wire Line
-	4750 1050 4750 1700
-Connection ~ 4750 1700
-Wire Wire Line
 	5550 1550 5550 1800
-Wire Wire Line
-	4750 1700 5350 1700
-Wire Wire Line
-	4700 1800 5550 1800
-Wire Wire Line
-	4500 950  4800 950
-Wire Wire Line
-	4800 950  4800 1600
-Wire Wire Line
-	4800 1600 4500 1600
-Wire Wire Line
-	4850 1600 4800 1600
-Connection ~ 4800 1600
-Text GLabel 3500 1200 2    50   Input ~ 0
-PWM0
-Text GLabel 3500 1300 2    50   Input ~ 0
-PWM1
 $Comp
 L Connector_Generic:Conn_01x07 J11
@@
 F 0 "J11" H 2700 550 50  0000 C CNN
 F 1 "Conn_01x07" H 2700 600 50  0000 C CNN
-F 2 "Connector_PinSocket_2.54mm:PinSocket_1x07_P2.54mm_Vertical" H 2800 1000 50  0001 C CNN
+F 2 "Connector_PinHeader_1.00mm:PinHeader_2x04_P1.00mm_Vertical_SMD" H 2800 1000 50  0001 C CNN
 F 3 "~" H 2800 1000 50  0001 C CNN
 	1    2800 1000
@@
 F 0 "J12" H 2700 1450 50  0000 C CNN
 F 1 "Conn_01x07" H 2700 1500 50  0000 C CNN
-F 2 "Connector_PinSocket_2.54mm:PinSocket_1x07_P2.54mm_Vertical" H 2800 1900 50  0001 C CNN
+F 2 "Connector_PinHeader_1.00mm:PinHeader_2x04_P1.00mm_Vertical_SMD" H 2800 1900 50  0001 C CNN
 F 3 "~" H 2800 1900 50  0001 C CNN
 	1    2800 1900
@@
 	3000 1100 3350 1100
 Wire Wire Line
-	3000 1200 3400 1200
-Wire Wire Line
 	3000 1600 3150 1600
 Wire Wire Line
@@
 Connection ~ 3350 1100
 Wire Wire Line
-	3400 1200 3400 2100
-Wire Wire Line
-	3400 2100 3000 2100
-Connection ~ 3400 1200
-Wire Wire Line
-	3000 1300 3450 1300
-Wire Wire Line
-	3400 1200 3500 1200
-Wire Wire Line
 	3350 1100 3500 1100
 Wire Wire Line
@@
 Wire Wire Line
 	3150 700  3500 700
-Wire Wire Line
-	3450 1300 3450 2200
-Wire Wire Line
-	3450 2200 3000 2200
-Connection ~ 3450 1300
-Wire Wire Line
-	3450 1300 3500 1300
 $Comp
 L Device:R_Small R29
@@
 	1    0    0    -1
 $EndComp
+$Comp
+L Connector_Generic:Conn_01x05 J4
+U 1 1 5EF1C02F
+P 4200 1800
+F 0 "J4" H 4200 1400 50  0000 C CNN
+F 1 "Conn_01x05" H 4250 1500 50  0000 C CNN
+F 2 "Connector_PinHeader_1.00mm:PinHeader_2x03_P1.00mm_Vertical_SMD" H 4200 1800 50  0001 C CNN
+F 3 "~" H 4200 1800 50  0001 C CNN
+	1    4200 1800
+	-1   0    0    1
+$EndComp
+Wire Wire Line
+	4400 1600 4650 1600
+Wire Wire Line
+	4400 1700 4600 1700
+Wire Wire Line
+	4400 1800 4550 1800
+Wire Wire Line
+	4400 1900 4500 1900
+Wire Wire Line
+	4400 2000 4450 2000
+$Comp
+L Connector_Generic:Conn_01x05 J1
+U 1 1 5EF40D9B
+P 4200 950
+F 0 "J1" H 4120 525 50  0000 C CNN
+F 1 "Conn_01x05" H 4120 616 50  0000 C CNN
+F 2 "Connector_PinHeader_1.00mm:PinHeader_2x03_P1.00mm_Vertical_SMD" H 4200 950 50  0001 C CNN
+F 3 "~" H 4200 950 50  0001 C CNN
+	1    4200 950
+	-1   0    0    1
+$EndComp
+Wire Wire Line
+	4400 1150 4450 1150
+Wire Wire Line
+	4450 1150 4450 2000
+Connection ~ 4450 2000
+Wire Wire Line
+	4450 2000 4650 2000
+Wire Wire Line
+	4500 1900 4500 1050
+Wire Wire Line
+	4500 1050 4400 1050
+Connection ~ 4500 1900
+Wire Wire Line
+	4500 1900 4850 1900
+Wire Wire Line
+	4400 950  4550 950
+Wire Wire Line
+	4550 950  4550 1800
+Connection ~ 4550 1800
+Wire Wire Line
+	4550 1800 5550 1800
+Wire Wire Line
+	4600 1700 4600 850
+Wire Wire Line
+	4600 850  4400 850
+Connection ~ 4600 1700
+Wire Wire Line
+	4600 1700 5350 1700
+Wire Wire Line
+	4400 750  4650 750
+Wire Wire Line
+	4650 750  4650 1600
+Connection ~ 4650 1600
+Wire Wire Line
+	4650 1600 4850 1600
+Text GLabel 4850 1900 2    50   Input ~ 0
+VBUS
+$Comp
+L power:GNDD #PWR?
+U 1 1 5EF5FD4C
+P 4650 2050
+AR Path="/5EF5FD4C" Ref="#PWR?"  Part="1"
+AR Path="/5E247314/5EF5FD4C" Ref="#PWR0101"  Part="1"
+F 0 "#PWR0101" H 4650 1800 50  0001 C CNN
+F 1 "GNDD" H 4500 2000 50  0000 C CNN
+F 2 "" H 4650 2050 50  0001 C CNN
+F 3 "" H 4650 2050 50  0001 C CNN
+	1    4650 2050
+	1    0    0    -1
+$EndComp
+NoConn ~ 3000 2100
+NoConn ~ 3000 2200
+NoConn ~ 3000 1300
+NoConn ~ 3000 1200
 Wire Bus Line
 	1550 5550 1550 5950

Commit message: 一歩進んで仕様決めなおし
Parts:
- removed C28, C31: 10n, micelib:C_0201_0603Metric_HandSoldering, symbol Device:C_Small
- removed C29, C30, C32, C33: 0.1u, micelib:C_0402_1005Metric_HandSoldering, symbol Device:C_Small
- removed R29: 10k, micelib:C_0402_1005Metric_HandSoldering, symbol Device:R_Small
- removed U10, U11: MPU-9250, micelib:InvenSense_QFN-24_3x3mm_P0.4mm_HandSoldering, symbol Sensor_Motion:MPU-9250
- added C? (x2): 0.1u, micelib:C_0402_1005Metric_HandSoldering, symbol Device:C_Small
- added J?: Conn_I2C, Connector_PinHeader_2.54mm:PinHeader_1x04_P2.54mm_Vertical, symbol Connector_Generic:Conn_01x04
- added J?: Conn_SPI, symbol Connector_Generic:Conn_01x05
Connections:
- net +3V3: now also C?.1, C?.1, J?.3 (Pin_3), J?.4 (Pin_4)
- net GNDD: now also C?.2, C?.2, J?.4 (Pin_4), J?.5 (Pin_5)
- net I2C_SCL: now also J?.1 (Pin_1)
- net I2C_SDA: now also J?.2 (Pin_2)
- net VSPI_CLK: now also J?.1 (Pin_1)
- net VSPI_MISO: now also J?.3 (Pin_3)
- net VSPI_MOSI: now also J?.2 (Pin_2)
- no-connect marks 14 -> 4
Other:
- note added: "I2C & SPI"
- note removed: "IMU"
- moved on the sheet: C22, J1, J11, J12, J4, R11, R27, R28, U9

Commit message: ちょっとシンプルにしよう
Parts:
- removed J11, J12: Conn_01x07, Connector_PinHeader_1.00mm:PinHeader_2x04_P1.00mm_Vertical_SMD, symbol Connector_Generic:Conn_01x07
- added J10: Conn_I2CBridge, symbol Connector_Generic:Conn_01x02
- added J9: Conn__I2CBridge, symbol Connector_Generic:Conn_01x02
- J11: renamed from J1; value Conn_01x05 -> Conn_PBridge
- J12: renamed from J4; value Conn_01x05 -> Conn__PBridge
- gave numbers to parts that had none: 4
- renumbered C22 to C19, R11 to R33, R27 to R34, R28 to R35, U9 to U8
Connections:
- net I2C_SCL: now also J10.1 (Pin_1), J9.1 (Pin_1)
- net I2C_SDA: now also J10.2 (Pin_2), J9.2 (Pin_2)
- net VSPI_CLK renamed SPI_CLK
- net VSPI_MISO renamed SPI_MISO
- net VSPI_MOSI renamed SPI_MOSI
- no-connect marks 4 -> 0
Other:
- note added: "Board_Bridge"
- moved on the sheet: C19, J11, J12, R33, R34, R35, U8

Commit message: Change MD to DRV8830
Parts:
- J10, J9: footprint (none) -> Connector_PinHeader_1.00mm:PinHeader_2x03_P1.00mm_Vertical_SMD
- J8: footprint (none) -> Connector_PinSocket_2.54mm:PinSocket_1x05_P2.54mm_Vertical
Changed lines of the file:
@@
 F 0 "J9" H 2970 1125 50  0000 C CNN
 F 1 "Conn__I2CBridge" H 2970 1216 50  0000 C CNN
-F 2 "" H 3050 1450 50  0001 C CNN
+F 2 "Connector_PinHeader_1.00mm:PinHeader_2x03_P1.00mm_Vertical_SMD" H 3050 1450 50  0001 C CNN
 F 3 "~" H 3050 1450 50  0001 C CNN
 	1    3050 1450
@@
 F 0 "J10" H 2970 1575 50  0000 C CNN
 F 1 "Conn_I2CBridge" H 2970 1666 50  0000 C CNN
-F 2 "" H 3050 1900 50  0001 C CNN
+F 2 "Connector_PinHeader_1.00mm:PinHeader_2x03_P1.00mm_Vertical_SMD" H 3050 1900 50  0001 C CNN
 F 3 "~" H 3050 1900 50  0001 C CNN
 	1    3050 1900
@@
 F 0 "J8" V 2316 2362 50  0000 R CNN
 F 1 "Conn_SPI" V 2225 2362 50  0000 R CNN
-F 2 "" H 2350 2650 50  0001 C CNN
+F 2 "Connector_PinSocket_2.54mm:PinSocket_1x05_P2.54mm_Vertical" H 2350 2650 50  0001 C CNN
 F 3 "~" H 2350 2650 50  0001 C CNN
 	1    2350 2650
